File: PCB Files/TobiV3 Aruino Version/tobi_arduino_version.brd (EAGLE design)
At the start: 103 x 74 mm, 45 parts

Commit message: let's try this again
Parts:
- added R_PB_LED: 1000, resistor:0204V
- R_LED0, R_LED1, R_LED2, R_LED3, R_LED4, R_LED5: value (none) -> 1000
- R_SCL, R_SDA: value (none) -> 100000
- moved H3 176.8 mm to (156.0, 95.0), turned to 270 degrees
- moved DRIVER2 123.8 mm to (129.8, 65.2)
- moved H4 91.5 mm to (61.2, 94.7), turned to 0 degrees
- moved PCF2 89.0 mm to (124.9, 53.1)
- moved DRIVER1 77.4 mm to (124.7, 76.5), turned to 90 degrees
- moved PCF1 77.4 mm to (96.9, 90.7), turned to 90 degrees
- moved R_LED2 75.4 mm to (68.6, 84.3)
- moved H1 75.0 mm to (61.0, 30.0), turned to 0 degrees
- moved H2 75.0 mm to (156.0, 30.0)
- moved R_LED4 73.4 mm to (68.4, 64.3)
- moved R_LED1 71.4 mm to (122.2, 96.3)
- moved R_LED5 71.0 mm to (155.7, 53.3)
- moved LED2 67.4 mm to (61.0, 85.1)
- moved PB_LED 66.8 mm to (147.7, 96.3)
- moved MOT_3 66.8 mm to (155.8, 86.7)
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Connections:
- removed net N$2: LED1.A, R_LED1.1
- removed net N$3: LED2.A, R_LED2.1
- removed net N$4: LED3.A, R_LED3.1
- removed net N$5: LED4.A, R_LED4.1
- removed net N$6: LED5.A, R_LED5.1
- net GND: no longer LED0.K, LED1.K, LED2.K, LED3.K, LED4.K, LED5.K, PB_LED.2
- net LED0: now also LED0.K, R_LED0.1
- net LED1: now also LED1.K, R_LED1.1
- net LED2: now also LED2.K, R_LED2.1
- net LED3: now also LED3.K, R_LED3.1
- net LED4: now also LED4.K, R_LED4.1
- net LED5: now also LED5.K, R_LED5.1
- net N$1: now also PB_LED.2, R_PB_LED.2; no longer LED0.A, R_LED0.1
- net PB_LED: now also R_PB_LED.1; no longer PB_LED.1
- net SCL: now also R_SCL.1; no longer R_SCL.2
- net SDA: now also R_SDA.1; no longer R_SDA.2
- net VCC: now also LED0.A, LED1.A, LED2.A, LED3.A, LED4.A, LED5.A, PB_LED.1, R_SCL.2, R_SDA.2; no longer R_SCL.1, R_SDA.1
Routing:
- net VCC: track 335.5 -> 0.00 mm, vias 1 -> 0
- net M5_PWM: track 132.9 -> 0.00 mm, vias 1 -> 0
- net M4_A: track 129.9 -> 0.00 mm, vias 4 -> 0
- net V_MOT: track 184.1 -> 65.4 mm, vias 7 -> 1
- net M3_PWM: track 107.2 -> 0.00 mm, vias 2 -> 0
- net LED4: track 105.8 -> 0.00 mm, vias 2 -> 0
- net M2_PWM: track 104.9 -> 0.00 mm, vias 4 -> 0
- net M4_B: track 102.4 -> 0.00 mm, vias 2 -> 0
- net SDA: track 98.5 -> 0.00 mm, vias 2 -> 0
- net RESET: track 97.1 -> 0.00 mm, vias 2 -> 0
- net M3_B: track 94.7 -> 0.00 mm, vias 5 -> 0
- net SCL: track 93.1 -> 0.00 mm, vias 3 -> 0
- net M3_A: track 90.1 -> 0.00 mm, vias 3 -> 0
- net MOSI: track 85.9 -> 0.00 mm, vias 2 -> 0
- net M0_ENC: track 80.2 -> 0.00 mm, vias 1 -> 0
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Other:
- board text added: "off"
- board text added: "on"
- board text removed: "OFF"
- board text removed: "ON"
- board text removed: "TOBI v4 Tom Dodson"
- board text removed: "www.grasp.upenn.edu"

Commit message: no routing
Routing:
- net V_MOT: track 65.4 -> 0.00 mm, vias 1 -> 0
- net V_BATT: track 17.2 -> 0.00 mm
Changed lines of the file:
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@@
 </variantdefs>
 <classes>
-<class number="0" name="default" width="0" drill="0">
+<class number="0" name="default" width="0.4064" drill="0">
+<clearance class="0" value="0.2032"/>
 </class>
 </classes>
@@
 <param name="RoutingGrid" value="50mil"/>
 <param name="AutoGrid" value="1"/>
-<param name="Efforts" value="0"/>
+<param name="Efforts" value="2"/>
 <param name="TopRouterVariant" value="1"/>
 <param name="tpViaShape" value="round"/>
@@
 <contactref element="C1" pad="1"/>
 <contactref element="SWITCH" pad="P"/>
-<wire x1="73.58" y1="36.48" x2="69.63" y2="32.53" width="0.4064" layer="1"/>
-<wire x1="69.63" y1="32.53" x2="69.63" y2="31.39" width="0.4064" layer="1"/>
-<wire x1="69.63" y1="31.39" x2="63.6938" y2="37.3262" width="0.4064" layer="1"/>
-<wire x1="63.6938" y1="37.3262" x2="63.6938" y2="38.07449375" width="0.4064" layer="1"/>
-<wire x1="62.5" y1="39.26829375" x2="62.5" y2="40.12" width="0.4064" layer="1"/>
-<wire x1="63.6938" y1="38.07449375" x2="62.5" y2="39.26829375" width="0.4064" layer="1"/>
 <wire x1="120.92" y1="77.72" x2="131.06" y2="69.02" width="0" layer="19" extent="1-1"/>
 <wire x1="110.52" y1="65.93" x2="120.92" y2="77.72" width="0" layer="19" extent="1-1"/>
 <wire x1="130.55" y1="46.02" x2="131.06" y2="69.02" width="0" layer="19" extent="1-1"/>
 <wire x1="86.64" y1="76.76" x2="110.52" y2="65.93" width="0" layer="19" extent="1-1"/>
-<wire x1="91" y1="75" x2="86.64" y2="76.76" width="0" layer="19" extent="1-16"/>
-<via x="91" y="75" extent="1-16" drill="0.35"/>
-<wire x1="73.58" y1="36.48" x2="84.7604" y2="47.6604" width="0.4064" layer="16"/>
-<wire x1="84.7604" y1="47.6604" x2="84.7604" y2="49.28293125" width="0.4064" layer="16"/>
-<wire x1="84.7604" y1="49.28293125" x2="85.71986875" y2="50.2424" width="0.4064" layer="16"/>
-<wire x1="85.71986875" y1="50.2424" x2="87.86493125" y2="50.2424" width="0.4064" layer="16"/>
-<wire x1="87.86493125" y1="50.2424" x2="91" y2="53.37746875" width="0.4064" layer="16"/>
-<wire x1="91" y1="53.37746875" x2="91" y2="75" width="0.4064" layer="16"/>
+<wire x1="73.58" y1="36.48" x2="86.64" y2="76.76" width="0" layer="19" extent="1-1"/>
+<wire x1="69.63" y1="31.39" x2="73.58" y2="36.48" width="0" layer="19" extent="1-1"/>
+<wire x1="62.5" y1="40.12" x2="69.63" y2="31.39" width="0" layer="19" extent="1-1"/>
 </signal>
 <signal name="M0_A">
@@
 <contactref element="POWR-PLUG" pad="POW"/>
 <contactref element="SWITCH" pad="O"/>
-<wire x1="66.36" y1="50.29" x2="64.2406" y2="48.1706" width="0.4064" layer="1"/>
-<wire x1="64.2406" y1="48.1706" x2="64.2406" y2="47.81770625" width="0.4064" layer="1"/>
-<wire x1="64.2406" y1="47.81770625" x2="59" y2="42.57710625" width="0.4064" layer="1"/>
-<wire x1="59" y1="41.08" x2="62.5" y2="37.58" width="0.4064" layer="1"/>
-<wire x1="59" y1="42.57710625" x2="59" y2="41.08" width="0.4064" layer="1"/>
+<wire x1="62.5" y1="37.58" x2="66.36" y2="50.29" width="0" layer="19" extent="1-1"/>
 </signal>
 <signal name="N$1">
