File: PCB Files/TobiV3 Aruino Version/tobi_arduino_version.sch (EAGLE design)
At the start: 56 parts, among them M1 M1_M2, M2 M1_M2, M3 DF11-4PIN, M4 DF11-4PIN, M5 DF11-4PIN, M6 DF11-4PIN

Commit message: try to use the old pcb
Parts:
- removed EXTERNALSWITCH: M02PTH, SparkFun-Connectors:M02PTH
- removed M1, M2: M1_M2, Gavin:DF11-4PIN
- removed M3, M4, M5, M6: DF11-4PIN, Gavin:DF11-4PIN
- added MOT1, MOT2, MOT3, MOT4, MOT5, MOT6: (no value), pinhead:PINHD-1X2
- ENC1, ENC2, ENC3, ENC4, ENC5, ENC6: value DF11-4PIN -> (none); device Gavin:DF11-4PIN -> pinhead:PINHD-1X3
Connections:
- removed net D12: ARDUINOMICRO.12, JP1.11
- removed net V_IN_1: EXTERNALSWITCH.2, SWITCH.P
- new net D13: ARDUINOMICRO.13, JP1.11
- net GND: now also ENC1.2, ENC2.2, ENC3.2, ENC4.2, ENC5.2, ENC6.2; no longer ENC1.P2, ENC2.P2, ENC3.P2, ENC4.P2, ENC5.P2, ENC6.P2
- net M1_A: now also MOT1.1; no longer M1.P1
- net M1_B: now also MOT1.2; no longer M1.P2
- net M1_ENC: now also ENC1.3; no longer ENC1.P3
- net M2_A: now also MOT2.1; no longer M2.P1
- net M2_B: now also MOT2.2; no longer M2.P2
- net M2_ENC: now also ENC2.3; no longer ENC2.P3
- net M3_A: now also MOT3.1; no longer M3.P1
- net M3_B: now also MOT3.2; no longer M3.P2
- net M3_ENC: now also ENC3.3; no longer ENC3.P3
- net M4_A: now also MOT4.1; no longer M4.P1
- net M4_B: now also MOT4.2; no longer M4.P2
- net M4_ENC: now also ENC4.3; no longer ENC4.P3
- net M5_A: now also MOT5.1; no longer M5.P1
- net M5_B: now also MOT5.2; no longer M5.P2
- net M5_ENC: now also ENC5.3; no longer ENC5.P3
- net M6_A: now also MOT6.1; no longer M6.P1
- net M6_B: now also MOT6.2; no longer M6.P2
- net M6_ENC: now also ENC6.3; no longer ENC6.P3
- net M6_PWM: now also ARDUINOMICRO.12; no longer ARDUINOMICRO.13
- net VCC: now also ENC1.1, ENC2.1, ENC3.1, ENC4.1, ENC5.1, ENC6.1; no longer ARDUINOMICRO.9V, ENC1.P1, ENC2.P1, ENC3.P1, ENC4.P1, ENC5.P1, ENC6.P1
- net V_IN: now also ARDUINOMICRO.9V, SWITCH.P; no longer EXTERNALSWITCH.1
Other:
- note removed: "M1_M2"
